File: boards/prom-shield/prom-shield.kicad_pcb (KiCad board)
At the start: 2 copper layers, 68.6 x 53.3 mm, 8 parts, among them J1 Power, J2 Digital/PWM, J3 Analog, J4 Digital/PWM

Commit message: Initial PCB revision for ROM programmer
Parts:
- added C1: 0.1 µF, Capacitor_THT:C_Disc_D5.0mm_W2.5mm_P5.00mm, F.Cu at (102.3, 58.5)
- added C2: 0.1 µF, Capacitor_THT:C_Disc_D5.0mm_W2.5mm_P5.00mm, F.Cu at (143.0, 92.2)
- added C3: 0.1 µF, Capacitor_THT:C_Disc_D5.0mm_W2.5mm_P5.00mm, F.Cu at (157.0, 64.0)
- added R1: 10 kΩ, Resistor_THT:R_Axial_DIN0207_L6.3mm_D2.5mm_P7.62mm_Horizontal, F.Cu at (111.2, 58.5)
- added R2: 10 kΩ, Resistor_THT:R_Axial_DIN0207_L6.3mm_D2.5mm_P7.62mm_Horizontal, F.Cu at (121.7, 58.5)
- added R3: 10 kΩ, Resistor_THT:R_Axial_DIN0207_L6.3mm_D2.5mm_P7.62mm_Horizontal, F.Cu at (132.7, 58.5)
- added U1: 28C256, Socket:DIP_Socket-28_W11.9mm_W12.7mm_W15.24mm_W17.78mm_W18.5mm_3M_228-1277-00-0602J, F.Cu at (112.3, 80.0)
- added U2: 74HC595, Package_DIP:DIP-16_W7.62mm_Socket_LongPads, F.Cu at (133.9, 86.2)
- added U3: 74HC595, Package_DIP:DIP-16_W7.62mm_Socket_LongPads, F.Cu at (155.7, 68.9)
- renumbered J3 to J1, J1 to J2, J2 to J3
Connections:
- J1 pad 1: /A0 -> /~{WE}
- J1 pad 2: /A1 -> /~{CE}
- J1 pad 3: /A2 -> /~{OE}
- J1 pad 4: /A3 -> /USR_SRCLK
- J1 pad 5: /SDA/A4 -> /LSR_SRCLK
- J1 pad 6: /SCL/A5 -> /SER
- J2 pad 2: /IOREF -> unconnected-(J2-IOREF-Pad2)
- J2 pad 3: /~{RESET} -> unconnected-(J2-~{RESET}-Pad3)
- J2 pad 4: +3V3 -> unconnected-(J2-3.3V-Pad4)
- J2 pad 5: +5V -> VCC
- J2 pad 8: VCC -> unconnected-(J2-Vin-Pad8)
- J3 pad 1: /SCL/A5 -> unconnected-(J3-SCL-Pad1)
- J3 pad 10: /8 -> /D6
- J3 pad 2: /SDA/A4 -> unconnected-(J3-SDA-Pad2)
- J3 pad 3: /AREF -> unconnected-(J3-AREF-Pad3)
- J3 pad 5: /13 -> /RCLK
- J3 pad 6: /12 -> unconnected-(J3-12-Pad6)
- J3 pad 7: /*11 -> unconnected-(J3-~11-Pad7)
- J3 pad 8: /*10 -> unconnected-(J3-~10-Pad8)
- J3 pad 9: /*9 -> /D7
- J4 pad 1: /7 -> /D5
- J4 pad 2: /*6 -> /D4
- J4 pad 3: /*5 -> /D3
- J4 pad 4: /4 -> /D2
- J4 pad 5: /*3 -> /D1
- J4 pad 6: /2 -> /D0
- J4 pad 7: /TX/1 -> unconnected-(J4-TX/1-Pad7)
- J4 pad 8: /RX/0 -> unconnected-(J4-RX/0-Pad8)
Routing:
- net VCC: track 0.00 -> 160.9 mm, vias 0 -> 6
- net /RCLK: track 0.00 -> 84.8 mm, vias 0 -> 3
- net /~{WE}: track 0.00 -> 64.5 mm, vias 0 -> 2
- net /SER: track 0.00 -> 62.5 mm
- net /~{OE}: track 0.00 -> 58.2 mm, vias 0 -> 2
- net /~{CE}: track 0.00 -> 56.4 mm, vias 0 -> 2
- net /A8: track 0.00 -> 50.7 mm
- net /A13: track 0.00 -> 50.5 mm, vias 0 -> 4
- net /D0: track 0.00 -> 50.0 mm, vias 0 -> 2
- net /A14: track 0.00 -> 48.8 mm
- net /A11: track 0.00 -> 46.5 mm
- net /LSR_SRCLK: track 0.00 -> 44.9 mm
- net /D1: track 0.00 -> 44.1 mm, vias 0 -> 2
- net /A12: track 0.00 -> 42.3 mm
- net /D2: track 0.00 -> 35.9 mm, vias 0 -> 2
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- added copper zone on B.Cu, net GND
Other:
- rule pad_to_mask_clearance: 0 -> 0.1
